File: Hardware/TapTempoPCB_V1_KiCad/TapTempo.sch (KiCad schematic (older format))
At the start: 10 parts, among them Q1 PN2222A, SW1 SPST, U1 PIC12F1822

Commit message: Added the DAC and cleaned up the schematic a little bit.
Parts:
- removed C1: Csmall, symbol Csmall
- added C? (x2): C, ~, symbol C
- added P?: CONN_1, symbol CONN_1
- added P?: CONN_2, symbol CONN_2
- added P?: CONN_6, symbol CONN_6
- added R? (x2): 4.7K, ~, symbol R
- added RV?: POT, symbol POT
- added U?: MCP4725, SOT-23-6, symbol MCP4725
- Q1: value PN2222A -> 2N3904
Connections:
- net labels added: TAP
- net labels removed: GateOut, TAP_IN
- wire segments 39 -> 66
Other:
- note added: "DAC"
- note added: "FTDI"
- note added: "GATE & TAP INPUT"
- note added: "MICRO\n"
- note added: "POWER"
- note added: "PROGRAMMING"
- note added: "TIME KNOB"

Commit message: Anotation of schematic plus initial parts selection
Parts:
- added P4: CONN_1, symbol CONN_1
- gave numbers to parts that had none: 13
- renumbered U1 to U2
Connections:
- net Gatein: now also R1.1, P4.1; no longer R1.2
- net at Q1.1 (B): now also R1.2; no longer R1.1
- no-connect marks 0 -> 3

Commit message: Added LUT table to firmware for VCO also added spreadsheet for LUT
Parts:
- C1, C3: value C -> .1uF; footprint ~ -> Capacitors_SMD:C_1206_HandSoldering
- C2: footprint ~ -> Capacitors_SMD:C_1206_HandSoldering
- D1: footprint ~ -> Diodes_SMD:Diode-SMA_Standard
- P1: footprint (none) -> Connect:SIL-2
- P2: footprint (none) -> Connect:SIL-5
- P3: footprint (none) -> Connect:SIL-6
- P4, P5: footprint (none) -> Connect:SIL-1
- Q1: footprint TO92 -> Transistors_SMD:sot23
- R1, R2: footprint (none) -> Resistors_SMD:R_1206_HandSoldering
- R3, R4, R5: footprint ~ -> Resistors_SMD:R_1206_HandSoldering
- RV1: footprint (none) -> Potentiometers:Potentiometer_Triwood_RM-065
- SW1: footprint (none) -> Discret:SW_PUSH_SMALL
- U1: footprint SOT-23-6 -> SMD_Packages:SOT-23-6
- U2: footprint ~ -> SMD_Packages:SOIC-8-W
Changed lines of the file:
@@
 LIBS:valves
 LIBS:mcp4725
+LIBS:My_Library
 LIBS:TapTempo-cache
-EELAYER 27 0
+EELAYER 25 0
 EELAYER END
 $Descr A4 11693 8268
@@
 F 0 "U2" H 8750 2350 60  0000 C CNN
 F 1 "PIC12F1822" H 8800 3100 60  0000 C CNN
-F 2 "~" H 8800 2350 60  0000 C CNN
+F 2 "SMD_Packages:SOIC-8-W" H 8800 2350 60  0000 C CNN
 F 3 "" H 8800 2350 60  0000 C CNN
 	1    8800 2350
@@
 F 0 "Q1" H 2500 6102 40  0000 R CNN
 F 1 "2N3904" H 2500 6400 40  0000 R CNN
-F 2 "TO92" H 2400 6352 29  0001 C CNN
+F 2 "Transistors_SMD:sot23" H 2400 6352 29  0001 C CNN
 F 3 "" H 2500 6250 60  0000 C CNN
 	1    2500 6250
@@
 F 0 "R2" V 3230 5550 40  0000 C CNN
 F 1 "100K" V 3157 5551 40  0000 C CNN
-F 2 "" V 3080 5550 30  0000 C CNN
+F 2 "Resistors_SMD:R_1206_HandSoldering" V 3080 5550 30  0001 C CNN
 F 3 "" H 3150 5550 30  0000 C CNN
 	1    3150 5550
@@
 F 0 "SW1" H 3150 6600 70  0000 C CNN
 F 1 "SPST" H 3150 6400 70  0000 C CNN
-F 2 "" H 3150 6500 60  0000 C CNN
+F 2 "Discret:SW_PUSH_SMALL" H 3150 6500 60  0001 C CNN
 F 3 "" H 3150 6500 60  0000 C CNN
 	1    3150 6500
@@
 F 0 "R3" V 4330 5650 40  0000 C CNN
 F 1 "4.7K" V 4257 5651 40  0000 C CNN
-F 2 "~" V 4180 5650 30  0000 C CNN
+F 2 "Resistors_SMD:R_1206_HandSoldering" V 4180 5650 30  0000 C CNN
 F 3 "~" H 4250 5650 30  0000 C CNN
 	1    4250 5650
@@
 F 0 "D1" H 4250 6000 40  0000 C CNN
 F 1 "DIODE" H 4250 5800 40  0000 C CNN
-F 2 "~" H 4250 5900 60  0000 C CNN
+F 2 "Diodes_SMD:Diode-SMA_Standard" H 4250 5900 60  0000 C CNN
 F 3 "~" H 4250 5900 60  0000 C CNN
 	1    4250 5900
@@
 F 0 "C2" H 4700 6550 40  0000 L CNN
 F 1 ".1uF" H 4706 6365 40  0000 L CNN
-F 2 "~" H 4738 6300 30  0000 C CNN
+F 2 "Capacitors_SMD:C_1206_HandSoldering" H 4738 6300 30  0000 C CNN
 F 3 "~" H 4700 6450 60  0000 C CNN
 	1    4700 6450
@@
 F 0 "P2" V 1200 2550 50  0000 C CNN
 F 1 "CONN_5" V 1300 2550 50  0000 C CNN
-F 2 "" H 1250 2550 60  0000 C CNN
+F 2 "Connect:SIL-5" H 1250 2550 60  0001 C CNN
 F 3 "" H 1250 2550 60  0000 C CNN
 	1    1250 2550
@@
 L POT RV1
 U 1 1 545B75D4
-P 7600 6350
-F 0 "RV1" H 7600 6250 50  0000 C CNN
-F 1 "POT" H 7600 6350 50  0000 C CNN
-F 2 "" H 7600 6350 60  0000 C CNN
-F 3 "" H 7600 6350 60  0000 C CNN
-	1    7600 6350
+P 3950 3750
+F 0 "RV1" H 3950 3650 50  0000 C CNN
+F 1 "POT" H 3950 3750 50  0000 C CNN
+F 2 "Potentiometers:Potentiometer_Triwood_RM-065" H 3950 3750 60  0001 C CNN
+F 3 "" H 3950 3750 60  0000 C CNN
+	1    3950 3750
 	0    1    1    0
 $EndComp
@@
 L VCC #PWR03
 U 1 1 545B7899
-P 7600 5950
-F 0 "#PWR03" H 7600 6050 30  0001 C CNN
-F 1 "VCC" H 7600 6050 30  0000 C CNN
-F 2 "" H 7600 5950 60  0000 C CNN
-F 3 "" H 7600 5950 60  0000 C CNN
-	1    7600 5950
-	1    0    0    -1
-$EndComp
-Wire Wire Line
-	7600 6100 7600 5950
-Wire Wire Line
-	7600 6600 7600 6750
-Wire Wire Line
-	7750 6350 8000 6350
-Text GLabel 8000 6350 2    60   Input ~ 0
+P 3950 3350
+F 0 "#PWR03" H 3950 3450 30  0001 C CNN
+F 1 "VCC" H 3950 3450 30  0000 C CNN
+F 2 "" H 3950 3350 60  0000 C CNN
+F 3 "" H 3950 3350 60  0000 C CNN
+	1    3950 3350
+	1    0    0    -1
+$EndComp
+Wire Wire Line
+	3950 3500 3950 3350
+Wire Wire Line
+	3950 4000 3950 4150
+Wire Wire Line
+	4100 3750 4350 3750
+Text GLabel 4350 3750 2    60   Input ~ 0
 POT
 $Comp
@@
 F 0 "U1" H 8100 4900 40  0000 C CNN
 F 1 "MCP4725" H 8350 4850 40  0000 C CNN
-F 2 "SOT-23-6" H 8500 4550 30  0000 C CIN
+F 2 "SMD_Packages:SOT-23-6" H 8500 4550 30  0000 C CIN
 F 3 "" H 8650 4550 60  0000 C CNN
 	1    8650 4550
@@
 F 0 "R4" V 7830 3950 40  0000 C CNN
 F 1 "4.7K" V 7757 3951 40  0000 C CNN
-F 2 "~" V 7680 3950 30  0000 C CNN
+F 2 "Resistors_SMD:R_1206_HandSoldering" V 7680 3950 30  0000 C CNN
 F 3 "~" H 7750 3950 30  0000 C CNN
 	1    7750 3950
@@
 F 0 "R5" V 8380 3950 40  0000 C CNN
 F 1 "4.7K" V 8307 3951 40  0000 C CNN
-F 2 "~" V 8230 3950 30  0000 C CNN
+F 2 "Resistors_SMD:R_1206_HandSoldering" V 8230 3950 30  0000 C CNN
 F 3 "~" H 8300 3950 30  0000 C CNN
 	1    8300 3950
@@
 F 0 "P5" H 9880 4400 40  0000 L CNN
 F 1 "CONN_1" H 9800 4455 30  0001 C CNN
-F 2 "" H 9800 4400 60  0000 C CNN
+F 2 "Connect:SIL-1" H 9800 4400 60  0001 C CNN
 F 3 "" H 9800 4400 60  0000 C CNN
 	1    9800 4400
@@
 F 0 "P1" V 1200 1300 40  0000 C CNN
 F 1 "CONN_2" V 1300 1300 40  0000 C CNN
-F 2 "" H 1250 1300 60  0000 C CNN
+F 2 "Connect:SIL-2" H 1250 1300 60  0001 C CNN
 F 3 "" H 1250 1300 60  0000 C CNN
 	1    1250 1300
@@
 P 8750 1200
 F 0 "C3" H 8750 1300 40  0000 L CNN
-F 1 "C" H 8756 1115 40  0000 L CNN
-F 2 "~" H 8788 1050 30  0000 C CNN
+F 1 ".1uF" H 8756 1115 40  0000 L CNN
+F 2 "Capacitors_SMD:C_1206_HandSoldering" H 8788 1050 30  0000 C CNN
 F 3 "~" H 8750 1200 60  0000 C CNN
 	1    8750 1200
@@
 P 2000 1250
 F 0 "C1" H 2000 1350 40  0000 L CNN
-F 1 "C" H 2006 1165 40  0000 L CNN
-F 2 "~" H 2038 1100 30  0000 C CNN
+F 1 ".1uF" H 2006 1165 40  0000 L CNN
+F 2 "Capacitors_SMD:C_1206_HandSoldering" H 2038 1100 30  0000 C CNN
 F 3 "~" H 2000 1250 60  0000 C CNN
 	1    2000 1250
@@
 F 0 "P3" V 1250 4000 60  0000 C CNN
 F 1 "CONN_6" V 1350 4000 60  0000 C CNN
-F 2 "" H 1300 4000 60  0000 C CNN
+F 2 "Connect:SIL-6" H 1300 4000 60  0001 C CNN
 F 3 "" H 1300 4000 60  0000 C CNN
 	1    1300 4000
@@
 Text Notes 7850 5000 0    60   ~ 0
 DAC
-Text Notes 7850 6750 0    60   ~ 0
+Text Notes 4200 4150 0    60   ~ 0
 TIME KNOB
 Wire Notes Line
-	7000 5650 8800 5650
-Wire Notes Line
-	8800 5650 8800 7000
-Wire Notes Line
-	8800 7000 7000 7000
-Wire Notes Line
-	7000 7000 7000 5650
+	3350 3050 5150 3050
+Wire Notes Line
+	5150 3050 5150 4400
+Wire Notes Line
+	5150 4400 3350 4400
+Wire Notes Line
+	3350 4400 3350 3050
 Wire Notes Line
 	7150 3500 10200 3500
@@
 F 0 "R1" V 1780 6250 40  0000 C CNN
 F 1 "10K" V 1707 6251 40  0000 C CNN
-F 2 "" V 1630 6250 30  0000 C CNN
+F 2 "Resistors_SMD:R_1206_HandSoldering" V 1630 6250 30  0001 C CNN
 F 3 "" H 1700 6250 30  0000 C CNN
 	1    1700 6250
@@
 F 0 "P4" H 1380 6450 40  0000 L CNN
 F 1 "CONN_1" H 1300 6505 30  0001 C CNN
-F 2 "" H 1300 6450 60  0000 C CNN
+F 2 "Connect:SIL-1" H 1300 6450 60  0001 C CNN
 F 3 "" H 1300 6450 60  0000 C CNN
 	1    1300 6450
@@
 L GND #PWR013
 U 1 1 5462A795
-P 7600 6750
-F 0 "#PWR013" H 7600 6750 30  0001 C CNN
-F 1 "GND" H 7600 6680 30  0001 C CNN
-F 2 "" H 7600 6750 60  0000 C CNN
-F 3 "" H 7600 6750 60  0000 C CNN
-	1    7600 6750
-	1    0    0    -1
-$EndComp
+P 3950 4150
+F 0 "#PWR013" H 3950 4150 30  0001 C CNN
+F 1 "GND" H 3950 4080 30  0001 C CNN
+F 2 "" H 3950 4150 60  0000 C CNN
+F 3 "" H 3950 4150 60  0000 C CNN
+	1    3950 4150
+	1    0    0    -1
+$EndComp

Commit message: Lots of changes to the TapTempo Board, made it all consistantly surface mount, turned into a module and created gerbers.
Parts:
- removed P1: CONN_2, Connect:SIL-2, symbol CONN_2
- removed P2: CONN_5, Connect:SIL-5, symbol CONN_5
- removed P3: CONN_6, Connect:SIL-6, symbol CONN_6
- removed P5: CONN_1, Connect:SIL-1, symbol CONN_1
- removed RV1: POT, Potentiometers:Potentiometer_Triwood_RM-065, symbol POT
- removed SW1: SPST, Discret:SW_PUSH_SMALL, symbol SPST
- added C4: 1uF, Capacitors_SMD:C_1206_HandSoldering, symbol C
- added C5: .1uF, Capacitors_SMD:C_0805, symbol C
- added J1: ISPTOUCH_PIC, My_Library:ICSP_TOUCH_AVX_9188_6-WAY_MATING_GUIDE, symbol ISPTOUCH_PIC
- added P1: PWR, My_Library:Castellation, symbol CONN_1
- added P10: Low, My_Library:Castellation, symbol CONN_1
- added P11, P2: GND, My_Library:Castellation, symbol CONN_1
- added P3: CONN_01X02, Connect:PINHEAD1-2, symbol CONN_01X02
- added P4: DAC, My_Library:Castellation, symbol CONN_1
- added P6: Switch_1, My_Library:Castellation, symbol CONN_1
- added P7: Switch_2, My_Library:Castellation, symbol CONN_1
- added P8: High, My_Library:Castellation, symbol CONN_1
- added P9: Wiper, My_Library:Castellation, symbol CONN_1
- added U3: LDK220, Housings_SOT-23_SOT-143_TSOT-6:SOT-23-5, symbol LDK220
- C1: value .1uF -> 1uF
- C2, C3: footprint Capacitors_SMD:C_1206_HandSoldering -> Capacitors_SMD:C_0805
- D1: footprint Diodes_SMD:Diode-SMA_Standard -> Diodes_SMD:SOD-123
- P5: renamed from P4; value CONN_1 -> Gate; footprint Connect:SIL-1 -> My_Library:Castellation
- R1, R2, R3, R4, R5: footprint Resistors_SMD:R_1206_HandSoldering -> My_Library:R_0805
Connections:
- net GND: now also C4.1, C5.2, J1.6, P10.1, P11.1, P2.1, P3.1 (P1), P7.1, U3.2 (GND)
- net MCLR: now also J1.1
- net PGC: now also J1.5
- net PGD: now also J1.3, P3.2 (P2)
- net POT: now also C5.1, P9.1
- net VCC: now also C4.2, J1.2, P8.1, U3.5 (VOUT); no longer C1.2
- net at D1.1 (A), Q1.3 (C), R2.2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: now also P6.1
- net at U1.1 (Vout): now also P4.1
- new net: C1.2, P1.1, U3.1 (VIN), U3.3 (EN)
- no-connect marks 3 -> 1
